Commit message: Update puzzlebot_jetson_lidar_ed.xacro
Se cambio la refrerencia de paquete

File: urdf/mcr2_robots/puzzlebot_jetson_lidar_ed.xacro (robot description, xacro)
@@ -1,17 +1,23 @@
 <?xml version="1.0"?>
-<robot xmlns:xacro="http://www.ros.org/wiki/xacro" name="Puzzlebot_Jetson_Ed.">
-<xacro:arg name="prefix" default=""/>
-<!-- files for gazebo costumization -->
-<xacro:include filename="$(find m3_fampach)/urdf/mcr2_mechanical/puzzlebot_jetson_lidar_base.urdf.xacro"/>
-<xacro:include filename="$(find m3_fampach)/urdf/mcr2_robots/jetson_lidar_ed/parameters_jetson_lidar_ed.xacro" />
-<xacro:include filename="$(find m3_fampach)/urdf/mcr2_misc/materials.xacro" />
-<xacro:include filename="$(find m3_fampach)/urdf/mcr2_misc/macros.xacro" />
-<xacro:include filename="$(find m3_fampach)/urdf/mcr2_sensors/laser_camera_bracket.xacro" />
-<xacro:include filename="$(find m3_fampach)/urdf/mcr2_sensors/lidar.xacro" />
-<xacro:include filename="$(find m3_fampach)/urdf/mcr2_control/gazebo_control.xacro" />
-<!--LINKS-->
-<xacro:puzzlebot_jetson_lidar_ed_base prefix="$(arg prefix)" />
-<xacro:laser_camera_sensor prefix="$(arg prefix)" />
-<xacro:rpi_lidar_sensor prefix="$(arg prefix)" />
-<xacro:puzzlebot_control prefix="$(arg prefix)" />
+<robot xmlns:xacro="http://www.ros.org/wiki/xacro" name="puzzlebot_jetson_lidar_ed">
+  <!-- 1) Definimos el argumento prefix -->
+  <xacro:arg name="prefix" default=""/>
+  <!-- 2) Creamos una propiedad global para prefix -->
+  <xacro:property name="prefix" value="$(arg prefix)"/>
+  <!-- 3) Includes sin usar xacro:args -->
+  <xacro:include filename="$(find familiapachuquena_nav2_puzzlebot)/urdf/mcr2_mechanical/puzzlebot_jetson_lidar_base.urdf.xacro"/>
+  <xacro:include filename="$(find familiapachuquena_nav2_puzzlebot)/urdf/mcr2_robots/jetson_lidar_ed/parameters_jetson_lidar_ed.xacro"/>
+  <xacro:include filename="$(find familiapachuquena_nav2_puzzlebot)/urdf/mcr2_misc/materials.xacro"/>
+  <xacro:include filename="$(find familiapachuquena_nav2_puzzlebot)/urdf/mcr2_misc/macros.xacro"/>
+  <xacro:include filename="$(find familiapachuquena_nav2_puzzlebot)/urdf/mcr2_sensors/laser_camera_bracket.xacro"/>
+  <xacro:include filename="$(find familiapachuquena_nav2_puzzlebot)/urdf/mcr2_sensors/lidar.xacro"/>
+  <xacro:include filename="$(find familiapachuquena_nav2_puzzlebot)/urdf/mcr2_control/gazebo_control.xacro"/>
+  <!-- 4) Invocamos los macros / enlaces -->
+  <xacro:puzzlebot_jetson_lidar_ed_base prefix="${prefix}"/>
+  <xacro:laser_camera_sensor         prefix="${prefix}"/>
+  <xacro:rpi_lidar_sensor           prefix="${prefix}"
+                                    frame_name="laser_frame"
+                                    topic_name="scan"
+                                    update_rate="40"/>
+  <xacro:puzzlebot_control           prefix="${prefix}"/>
 </robot>
